File: hardware/kicad/system/current_sense.kicad_sch (KiCad schematic)
At the start: 17 parts, among them J1 kanal 1 retur, J2 kanal 2 retur, J3 kanal 3 retur, J4 Arduino, U1 LM358, U2 LM358

Commit message: Apply fiber-laser design rules from the DTU-PCB-prototyping guide
All seven boards rebuilt to meet the XTool fiber laser workflow
(SimsesLab/DTU-PCB-prototyping): 1.0 mm tracks, 0.8 mm clearance, solid
no-net fill zone on B.Cu (pad connection: none) so the laser only
engraves the isolation channels, DIP footprints switched to the
_LongPads variants from the guide's shop table.

TO packages cannot meet 0.8 mm pad-to-pad at stock sizes, so
energy_system.pretty now has TO-220-3_Vertical_LaserPads (pads narrowed
to 1.7 mm -> 0.84 mm gap; make_laserpads.py regenerates). The MPPT pass
transistor moves BD139 -> TIP41A (shop part): TO-126's 2.28 mm pitch can
never satisfy the rule, and TO-220 handles the ~7 W better anyway.

Two more bugs caught in this pass:
- Device:Q_NMOS uses letter pin numbers (G/D/S) while TO-220 pads are
  1/2/3 - buck/boost MOSFET pads silently got NO net in the earlier
  boards (no-net pads don't count as unconnected). pcb_build.py now maps
  G/D/S->1/2/3 and fails hard if a component ends up netless.
- DRC now 0 violations on all seven boards; remaining airwires are the
  documented jumpers.
Parts:
- U1, U2: footprint Package_DIP:DIP-8_W7.62mm -> Package_DIP:DIP-8_W7.62mm_LongPads
