File: hardware/kicad/system/system.kicad_pcb (KiCad board)
At the start: 2 copper layers, 200 x 130 mm, 131 parts, among them M501 IRF530, Q201 IRF540N, Q202 IRF530, Q401 IRF530, SW201 Switch, U201 LM7805, U202 MCP601, U203 NE555, U204 ILD74, U205 MCP601, U206 IR2110, U207 4N25, U208 IR2110, U301 MCP601, U302 IL300, U303 MCP601, U401 CNY17, U402 IR2110, U501 CNY17, U502 IR2110

Commit message: created complete pcb for whole system, ready for fabrication
Parts:
- moved C402 215.3 mm to (291.7, 146.9), turned to -90 degrees
- moved C209 211.8 mm to (260.7, 111.4), turned to -90 degrees
- moved J_STO101 208.3 mm to (224.7, 197.2)
- moved L401 200.3 mm to (240.3, 174.1), turned to 180 degrees
- moved U402 197.7 mm to (255.5, 176.2), turned to 180 degrees
- moved R402 189.7 mm to (270.2, 147.9), turned to 90 degrees
- moved U205 189.5 mm to (175.0, 147.3), turned to -90 degrees
- moved U206 188.8 mm to (206.9, 124.0), turned to 0 degrees
- moved U202 186.7 mm to (182.0, 140.9), turned to 180 degrees
- moved J_PV101 185.4 mm to (265.2, 77.9)
- moved U207 183.4 mm to (181.3, 154.4), turned to 90 degrees
- moved C405 178.6 mm to (261.2, 169.1), turned to -90 degrees
- moved D402 177.8 mm to (264.7, 133.4), turned to 90 degrees
- moved C201 174.9 mm to (151.5, 171.1)
- moved R401 174.8 mm to (269.0, 163.6), turned to 180 degrees
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Routing:
- net +5V_PWR: track 0.00 -> 663.9 mm, vias 0 -> 4
- net +15V_GATE: track 0.00 -> 567.2 mm, vias 0 -> 2
- net +15V2: track 0.00 -> 367.1 mm, vias 0 -> 1
- net GND_MCU: track 0.00 -> 322.4 mm, vias 0 -> 4
- net PWM_MOTOR: track 0.00 -> 260.6 mm, vias 0 -> 4
- net Net-(D203-K): track 0.00 -> 256.6 mm, vias 0 -> 3
- net PWM_BOOST: track 0.00 -> 235.8 mm, vias 0 -> 4
- net STORE: track 0.00 -> 191.7 mm
- net ADC_LOAD: track 0.00 -> 185.7 mm, vias 0 -> 4
- net LOAD: track 0.00 -> 150.2 mm, vias 0 -> 3
- net V1: track 0.00 -> 143.3 mm
- net ADC_V1: track 0.00 -> 129.7 mm, vias 0 -> 1
- net Net-(U206-LIN): track 0.00 -> 117.0 mm, vias 0 -> 3
- net SW: track 0.00 -> 107.0 mm
- net Net-(D205-K): track 0.00 -> 97.7 mm
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- added copper zone on B.Cu, net GND
- added copper zone on F.Cu, net GND
Other:
- board size 200 x 130 mm -> 220 x 133 mm
