File: hardware/kicad/boards/boost/boost.kicad_sch (KiCad schematic)
At the start: 11 parts, among them J1 lager ind (5V), J2 V2 ud (10V), J3 PWM (isoleret), J4 gate-forsyning, M1 IRF530, U1 4N25

Commit message: Assign G/D/S TO-220 footprint to Q_NMOS MOSFETs across boards (match symbol pins)
Parts:
- M1: footprint energy_system:TO-220-3_Vertical_LaserPads -> energy_system:TO-220-3_Vertical_LaserPads_GDS
