File: hardware/kicad/boards/boost/boost_v2/boost_v2.kicad_sch (KiCad schematic)
At the start: 17 parts, among them J1 lager ind (5V), J2 V2 ud (10V), J3 PWM (isoleret), J4 drive +15V, M1 IRF530, U1 CNY17, U2 IR2110

Commit message: Assign G/D/S TO-220 footprint to Q_NMOS MOSFETs across boards (match symbol pins)
Parts:
- M1: footprint energy_system:TO-220-3_Vertical_LaserPads -> energy_system:TO-220-3_Vertical_LaserPads_GDS
