File: hardware/kicad/boards/buck/buck.kicad_sch (KiCad schematic)
At the start: 11 parts, among them J1 V1 ind (15V), J2 5V ud, J3 PWM (isoleret), J4 gate-forsyning, M1 IRF530N, U1 4N25

Commit message: Assign G/D/S TO-220 footprint to Q_NMOS MOSFETs across boards (match symbol pins)
Parts:
- M1: footprint energy_system:TO-220-3_Vertical_LaserPads -> energy_system:TO-220-3_Vertical_LaserPads_GDS
